Commit message: working marker spawn in rviz, not sure about gazebo ``` cd experiment_ws catkin_make source experiment_ws/devel/setup.bash roslaunch marker classsim.launch ```

File: experiment_ws/src/marker/urdf/marker.urdf (robot description, URDF)
Before this commit: robot marker, 1 links, 0 joints
Links:
- link base_link: geometry visual mesh filename=package://marker/urdf/armarker_40.dae
